File: KiCad/TriCore-X/TriCore-X.kicad_sch (KiCad schematic)
At the start: 0 parts

Commit message: feat: design 5V and 12V power rails (schematic & PCB)
Other:
- added sheet Expansion_Port (Expansion_Port.kicad_sch)
Changed lines of the file:
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@@
 	(paper "A5")
+	(sheet
+		(at 54.61 17.78)
+		(size 31.75 15.24)
+		(exclude_from_sim no)
+		(in_bom yes)
+		(on_board yes)
+		(dnp no)
+		(fields_autoplaced yes)
+		(stroke
+			(width 0.1524)
+			(type solid)
+		)
+		(fill
+			(color 0 0 0 0.0000)
+		)
+		(property "Sheetname" "Expansion_Port"
+			(at 54.61 17.0684 0)
+			(effects
+				(font
+					(size 1.27 1.27)
+				)
+				(justify left bottom)
+			)
+		)
+		(property "Sheetfile" "Expansion_Port.kicad_sch"
+			(at 54.61 33.6046 0)
+			(effects
+				(font
+					(size 1.27 1.27)
+				)
+				(justify left top)
+			)
+		)
+		(instances
+			(project "TriCore-X"
+				(path "/b9ed8ff9-3a91-4311-b656-324fcf6f7e0c"
+					(page "7")
+				)
+			)
+		)
+	)
 	(sheet
 		(at 15.24 17.78)

Commit message: refactor: change core MCU to STM32H723 and add LPDDR4/HDMI support
Other:
- added sheet STM32 (STM32.kicad_sch)
Changed lines of the file:
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@@
+	)
+	(sheet
+		(at 54.61 41.91)
+		(size 31.75 15.24)
+		(exclude_from_sim no)
+		(in_bom yes)
+		(on_board yes)
+		(dnp no)
+		(fields_autoplaced yes)
+		(stroke
+			(width 0.1524)
+			(type solid)
+		)
+		(fill
+			(color 0 0 0 0.0000)
+		)
+		(property "Sheetname" "STM32"
+			(at 54.61 41.1984 0)
+			(effects
+				(font
+					(size 1.27 1.27)
+				)
+				(justify left bottom)
+			)
+		)
+		(property "Sheetfile" "STM32.kicad_sch"
+			(at 54.61 57.7346 0)
+			(effects
+				(font
+					(size 1.27 1.27)
+				)
+				(justify left top)
+			)
+		)
+		(instances
+			(project "TriCore-X"
+				(path "/b9ed8ff9-3a91-4311-b656-324fcf6f7e0c"
+					(page "8")
+				)
+			)
+		)
 	)
 	(sheet

Commit message: refactor: update schematic components and library references, including STM32H743 and new power symbols
Other:
- sheet RK3568B2 renamed MPU
- removed sheet DDR4
- sheet MPU: file RK3568B2.kicad_sch -> MPU.kicad_sch
Changed lines of the file:
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@@
-	)
-	(sheet
-		(at 15.24 66.04)
-		(size 31.75 15.24)
-		(exclude_from_sim no)
-		(in_bom yes)
-		(on_board yes)
-		(dnp no)
-		(fields_autoplaced yes)
-		(stroke
-			(width 0.1524)
-			(type solid)
-		)
-		(fill
-			(color 0 0 0 0.0000)
-		)
-		(property "Sheetname" "DDR4"
-			(at 15.24 65.3284 0)
-			(effects
-				(font
-					(size 1.27 1.27)
-				)
-				(justify left bottom)
-			)
-		)
-		(property "Sheetfile" "DDR4.kicad_sch"
-			(at 15.24 81.8646 0)
-			(effects
-				(font
-					(size 1.27 1.27)
-				)
-				(justify left top)
-			)
-		)
-		(instances
-			(project "TriCore-X"
-				(path "/b9ed8ff9-3a91-4311-b656-324fcf6f7e0c"
-					(page "4")
-				)
-			)
-		)
 	)
 	(sheet
@@
 			(color 0 0 0 0.0000)
 		)
-		(property "Sheetname" "RK3568B2"
+		(property "Sheetname" "MPU"
 			(at 15.24 41.1984 0)
 			(effects
@@
 			)
 		)
-		(property "Sheetfile" "RK3568B2.kicad_sch"
+		(property "Sheetfile" "MPU.kicad_sch"
 			(at 15.24 57.7346 0)
 			(effects
@@
 	)
 	(sheet
-		(at 54.61 41.91)
+		(at 15.24 66.04)
 		(size 31.75 15.24)
 		(exclude_from_sim no)
@@
 		)
 		(property "Sheetname" "STM32"
-			(at 54.61 41.1984 0)
+			(at 15.24 65.3284 0)
 			(effects
 				(font
@@
 		)
 		(property "Sheetfile" "STM32.kicad_sch"
-			(at 54.61 57.7346 0)
+			(at 15.24 81.8646 0)
 			(effects
 				(font
