File: KiCad/TriCore-X/FPGA.kicad_sch (KiCad schematic)
At the start: 1 part, among them U2 XC7A35T-FGG484

Commit message: refactor: change core MCU to STM32H723 and add LPDDR4/HDMI support
Parts:
- removed U2: XC7A35T-FGG484, Package_BGA:BGA-484_23.0x23.0mm_Layout22x22_P1.0mm, symbol FPGA_Xilinx_Artix7:XC7A35T-FGG484
- added U2: XC7A100T-FGG484, Package_BGA:BGA-484_23.0x23.0mm_Layout22x22_P1.0mm, symbol FPGA_Xilinx_Artix7:XC7A100T-FGG484
Connections:
- net GND: now also U2.A11 (GND), U2.A12 (GND), U2.A2 (GND), U2.A22 (GND), U2.A3 (GND), U2.A5 (GND), U2.A7 (GND), U2.A9 (GND), U2.AA12 (GND), U2.AA2 (GND), U2.AA22 (GND), U2.AB19 (GND), U2.AB9 (GND), U2.B12 (GND), U2.B19 (GND), U2.B3 (GND), U2.C10 (GND), U2.C12 (GND), U2.C16 (GND), U2.C3 (GND), U2.C6 (GND), U2.D12 (GND), U2.D13 (GND), U2.D3 (GND), U2.D4 (GND), U2.D8 (GND), U2.E11 (GND), U2.E20 (GND), U2.E4 (GND), U2.E5 (GND), U2.E7 (GND), U2.E9 (GND), U2.F11 (GND), U2.F17 (GND), U2.F5 (GND), U2.G10 (GND), U2.G12 (GND), U2.G14 (GND), U2.G5 (GND), U2.G6 (GND), U2.G7 (GND), U2.G8 (GND), U2.G9 (GND), U2.H1 (GND), U2.H11 (GND), U2.H21 (GND), U2.H7 (GND), U2.H9 (GND), U2.J10 (GND), U2.J12 (GND), U2.J18 (GND), U2.J8 (GND), U2.K11 (GND), U2.K15 (GND), U2.K5 (GND), U2.K7 (GND), U2.L2 (GND), U2.L22 (GND), U2.L8 (GND), U2.M11 (GND), U2.M19 (GND), U2.M7 (GND), U2.N16 (GND), U2.N6 (GND), U2.N8 (GND), U2.P11 (GND), U2.P13 (GND), U2.P3 (GND), U2.P7 (GND), U2.P9 (GND), U2.R10 (GND), U2.R12 (GND), U2.R20 (GND), U2.R8 (GND), U2.T11 (GND), U2.T17 (GND), U2.T7 (GND), U2.T9 (GND), U2.U14 (GND), U2.U4 (GND), U2.V1 (GND), U2.V11 (GND), U2.V21 (GND), U2.W18 (GND), U2.W8 (GND), U2.Y15 (GND), U2.Y5 (GND)

Commit message: refactor: update schematic components, remove unused files, and add new LED and CH334P symbols
Parts:
- removed U2: XC7A100T-FGG484, Package_BGA:BGA-484_23.0x23.0mm_Layout22x22_P1.0mm, symbol FPGA_Xilinx_Artix7:XC7A100T-FGG484
- added U1: XC7A35T-CSG325, Package_BGA:Xilinx_CSG325, symbol FPGA_Xilinx_Artix7:XC7A35T-CSG325
Connections:
- net GND: now also U1.A1 (GND), U1.A11 (GND), U1.A18 (GND), U1.A5 (GND), U1.A7 (GND), U1.A8 (GND), U1.B18 (GND), U1.B3 (GND), U1.B7 (GND), U1.B8 (GND), U1.C15 (GND), U1.C2 (GND), U1.C6 (GND), U1.C7 (GND), U1.D12 (GND), U1.D3 (GND), U1.D4 (GND), U1.D7 (GND), U1.E2 (GND), U1.E6 (GND), U1.E7 (GND), U1.E9 (GND), U1.F10 (GND), U1.F16 (GND), U1.F4 (GND), U1.F6 (GND), U1.G1 (GND), U1.G11 (GND), U1.G13 (GND), U1.G5 (GND), U1.G6 (GND), U1.G7 (GND), U1.G9 (GND), U1.H10 (GND), U1.H12 (GND), U1.H3 (GND), U1.H4 (GND), U1.H5 (GND), U1.H6 (GND), U1.H8 (GND), U1.J1 (GND), U1.J11 (GND), U1.J13 (GND), U1.J17 (GND), U1.J2 (GND), U1.J3 (GND), U1.J7 (GND), U1.K12 (GND), U1.K14 (GND), U1.K4 (GND), U1.K8 (GND), U1.L1 (GND), U1.L11 (GND), U1.L13 (GND), U1.L7 (GND), U1.M12 (GND), U1.M18 (GND), U1.M8 (GND), U1.N11 (GND), U1.N13 (GND), U1.N15 (GND), U1.N5 (GND), U1.N7 (GND), U1.N9 (GND), U1.P12 (GND), U1.P2 (GND), U1.P8 (GND), U1.R9 (GND), U1.T16 (GND), U1.T6 (GND), U1.U13 (GND), U1.U3 (GND), U1.V1 (GND), U1.V10 (GND), U1.V18 (GND)
