File: KiCad/TriCore-X/power.kicad_sch (KiCad schematic)
At the start: 103 parts, among them J1 PJ-035DH, Q1 AOD407, U3 TPS56637RPAR, U4 TPS56637RPAR, U5 RK809-5, Y1 32.768KHZ

Commit message: refactor: update schematic components and library references, including STM32H743 and new power symbols
Parts:
- removed C21, C22, C23, C24, C25, C26, C27, C28, C41, C42, C43, C45: 1uF, Capacitor_SMD:C_0402_1005Metric, symbol Device:C
- removed C44, C46, C47, C48, C49, C50: 10uF, Capacitor_SMD:C_0402_1005Metric, symbol Device:C
- removed C51, C52, C53, C54, C55, C56, C57, C58, C59, C60: 22uF, Capacitor_SMD:C_0805_2012Metric, symbol Device:C
- removed C61, C62, C63: 100nF, Capacitor_SMD:C_0402_1005Metric, symbol Device:C
- removed L3, L4, L5, L6, L7: FNR6045SR47NT, L_6045:IND-SMD_L6.0-W6.0_FNR60XXS, symbol L_6045:FNR6045SR47NT
- removed R18: 82K, Resistor_SMD:R_0402_1005Metric, symbol Device:R
- removed R19: 120K, Resistor_SMD:R_0402_1005Metric, symbol Device:R
- removed R20, R21: 4.7K, Resistor_SMD:R_0402_1005Metric, symbol Device:R
- removed R22: 100K, Resistor_SMD:R_0402_1005Metric, symbol Device:R
- removed R23: 22K, Resistor_SMD:R_0402_1005Metric, symbol Device:R
- removed R24, R25, R26: 10K, Resistor_SMD:R_0402_1005Metric, symbol Device:R
- removed U5: RK809-5, RK809-5:QFN-68_L7.0-W7.0-P0.35-BL-EP5.5, symbol RK809-5:RK809-5
- removed Y1: 32.768KHZ, Crystal:Crystal_DS26_D2.0mm_L6.0mm_Vertical, symbol Device:Crystal
- added L3, L4, L5, L6: 1.5uH, Inductor_SMD:L_Bourns_SRP7028A_7.3x6.6mm, symbol Device:L
- added R31: 20K, Resistor_SMD:R_0402_1005Metric, symbol Device:R
- added R32, R33, R37: 30K, Resistor_SMD:R_0402_1005Metric, symbol Device:R
- added R34, R36: 15K, Resistor_SMD:R_0402_1005Metric, symbol Device:R
- added R35: 68K, Resistor_SMD:R_0402_1005Metric, symbol Device:R
- added R38: 51K, Resistor_SMD:R_0402_1005Metric, symbol Device:R
- added R39: 10K, Resistor_SMD:R_0402_1005Metric, symbol Device:R
- added U8: EA3059, EA3059QDR:VQFN-24_L4.0-W4.0-P0.50-TL-EP2.5, symbol EA3059QDR:EA3059
- C14, C4: value 0.1uF -> 100nF
- C29, C30, C31: value 1uF -> 10uF
- C32: value 1uF -> 0.1uF
- C33, C35, C37: value 1uF -> 220pF
- C34, C36, C40: value 1uF -> 22uF; footprint Capacitor_SMD:C_0402_1005Metric -> Capacitor_SMD:C_0805_2012Metric
- C38: value 2.2uF -> 22uF; footprint Capacitor_SMD:C_0402_1005Metric -> Capacitor_SMD:C_0805_2012Metric
- C39: value 2.2uF -> 220pF
Connections:
- net BUCK5 is gone; now on net +5V: C31.1
- net VLDO5 is gone; now on net +5V: C29.1
- net VLDO6 is gone; now on net +5V: C30.1
- net VLDO7 is gone; now on net +5V: C32.1
- net VLDO9 is gone; now on net +1V0: C34.1
- net +5V: now also R39.1, U8.11 (VIN1), U8.20 (VIN4), U8.23 (VIN3), U8.3 (VCC), U8.8 (VIN2)
- net 5V_OK: now also R39.2, U8.22 (EN3)
- net GND: now also C38.2, R32.2, R34.2, R36.2, R38.2, U8.1 (GND3), U8.13 (GND1), U8.18 (GND4), U8.25 (EP), U8.4 (AGND), U8.6 (GND2); no longer C33.2, C35.2, C37.2, C39.2
- net +1V8: now reaches C36.1
- net +1V8: now also C35.1, L4.2, R33.1
- net +3.3V: now reaches C37.1
- net +3.3V: now also C38.1, L5.2, R35.1
- net +0.95V: now reaches C39.1
- net +0.95V: now also C40.1, L6.2, R37.1
- net VLDO8 renamed +1V0
- net +1V0: now also L3.2, R31.1
- new net FB1: C33.2, R31.2, R32.1, U8.14 (FB1)
- new net FB2: C35.2, R33.2, R34.1, U8.5 (FB2)
- new net FB3: C37.2, R35.2, R36.1, U8.2 (FB3)
- new net FB4: C39.2, R37.2, R38.1, U8.17 (FB4)
- new net LX1: L3.1, U8.12 (LX1)
- new net LX2: L4.1, U8.7 (LX2)
- new net LX3: L5.1, U8.24 (LX3)
- new net LX4: L6.1, U8.19 (LX4)
- no-connect marks 7 -> 2

Commit message: refactor: update schematic components, remove unused files, and add new LED and CH334P symbols
Parts:
- removed L3, L4, L5, L6: 1.5uH, Inductor_SMD:L_Bourns_SRP7028A_7.3x6.6mm, symbol Device:L
- removed U8: EA3059, EA3059QDR:VQFN-24_L4.0-W4.0-P0.50-TL-EP2.5, symbol EA3059QDR:EA3059
- added C41, C42, C43, C44: 1uF, Capacitor_SMD:C_0402_1005Metric, symbol Device:C
- added C45, C46, C47, C48: 22uF, Capacitor_SMD:C_0805_2012Metric, symbol Device:C
- added D10, D6, D7, D8, D9: LED, LED_SMD:LED_0603_1608Metric, symbol Device:LED
- added L3, L4, L5, L6: FWP252012P-1R0ML, FWP252012P-1R0ML:IND-SMD_L2.5-W2.0_YXMBL252010P, symbol FWP252012P-1R0ML:FWP252012P-1R0ML
- added R40, R41, R42, R43, R44: 49.9R, Resistor_SMD:R_0402_1005Metric, symbol Device:R
- added R45, R46, R47, R48, R49, R50, R51, R52, R53, R54, R55, R56, R57: 30K, Resistor_SMD:R_0402_1005Metric, symbol Device:R
- added U10, U7, U8, U9: SY8843QWC, SY8843QWC:QFN-7_L1.5-W1.5-P0.45-BL_SILERGY_SY8842QWC, symbol SY8843QWC:SY8843QWC
- added U11: RT9013-18GB, RT9013-18GB:SOT-23-5_L3.0-W1.7-P0.95-LS2.8-BR, symbol RT9013-18GB:RT9013-18GB
- added U12: RT9013-12GB, RT9013-12GB:SOT-23-5_L3.0-W1.7-P0.95-LS2.8-BR, symbol RT9013-12GB:RT9013-12GB
- added U13, U14, U15, U16: TPS22966DPUR, TPS22966DPUR:WSON-14_L3.0-W2.0-P0.40-BL-EP, symbol TPS22966DPUR:TPS22966DPUR
- C29, C31: value 10uF -> 22uF; footprint Capacitor_SMD:C_0402_1005Metric -> Capacitor_SMD:C_0805_2012Metric
- C30: value 10uF -> 100nF
- C32: value 0.1uF -> 22uF; footprint Capacitor_SMD:C_0402_1005Metric -> Capacitor_SMD:C_0805_2012Metric
- C33, C39: value 220pF -> 100nF
- C35, C37: value 220pF -> 22uF; footprint Capacitor_SMD:C_0402_1005Metric -> Capacitor_SMD:C_0805_2012Metric
- C36: value 22uF -> 100nF; footprint Capacitor_SMD:C_0805_2012Metric -> Capacitor_SMD:C_0402_1005Metric
- R31: value 20K -> 68K
- R32: value 30K -> 20K
- R33, R37: value 30K -> 15K
- R34, R36: value 15K -> 30K
- R35: value 68K -> 30K
- R38: value 51K -> 20K
- R39: value 10K -> 30K
Connections:
- net +1V8: now also C43.1, U11.5 (VOUT); no longer C35.1, C36.1, R33.1
- net +3.3V: now also U13.13 (VOUT1), U13.14 (VOUT1), U14.4 (VBIAS); no longer C37.1, C38.1, R35.1
- net +5V: now also C33.1, C35.1, C36.1, C38.1, C39.1, U10.5 (IN), U7.5 (IN), U8.5 (IN), U9.5 (IN); no longer C29.1
- net 5V_OK: now also U7.4 (EN)
- net GND: now also C33.2, C35.2, C37.2, C39.2, R33.2, C41.2, C42.2, C43.2, C44.2, C45.2, C46.2, C47.2, C48.2, R40.2, R41.2, R42.2, R43.2, R44.2, R47.2, R49.1, R50.1, R51.1, R52.1, R53.2, R54.2, R55.2, R56.2, R57.2, U10.7 (GND), U11.2 (GND), U12.2 (GND), U7.7 (GND), U8.7 (GND), U9.7 (GND); no longer R32.2, R36.2
- removed net +0.95V: C39.1, C40.1, R37.1
- removed net +1V0: C33.1, C34.1, R31.1
- removed net FB1: C33.2, R31.2, R32.1
- removed net FB2: C35.2, R33.2, R34.1
- removed net FB3: C37.2, R35.2, R36.1
- removed net FB4: C39.2, R37.2, R38.1
- new net: R31.2, R33.1, U7.1 (FB)
- new net: L3.1, U7.6 (LX)
- new net: D7.1 (K), R41.1
- new net: R37.2, R47.1, U9.1 (FB)
- new net: R54.1, U9.4 (EN)
- new net: L5.1, U9.6 (LX)
- new net: R57.1, U12.3 (EN)
- new net: R35.2, R38.1, U10.1 (FB)
- new net: U15.1 (VIN1), U15.2 (VIN1)
- new net: U15.13 (VOUT1), U15.14 (VOUT1)
- new net: U15.6 (VIN2), U15.7 (VIN2)
- new net: U15.8 (VOUT2), U15.9 (VOUT2)
- new net: U13.6 (VIN2), U13.7 (VIN2)
- new net: U13.8 (VOUT2), U13.9 (VOUT2)
- new net: D9.1 (K), R43.1
- new net: R32.2, R34.1, U8.1 (FB)
- new net: R53.1, U8.4 (EN)
- new net: L4.1, U8.6 (LX)
- new net: D8.1 (K), R42.1
- new net: U14.1 (VIN1), U14.2 (VIN1)
- new net: U14.13 (VOUT1), U14.14 (VOUT1)
- new net: U14.6 (VIN2), U14.7 (VIN2)
- new net: U14.8 (VOUT2), U14.9 (VOUT2)
- new net: R56.1, U11.3 (EN)
- new net: U16.1 (VIN1), U16.2 (VIN1)
- new net: U16.13 (VOUT1), U16.14 (VOUT1)
- new net: U16.6 (VIN2), U16.7 (VIN2)
- new net: U16.8 (VOUT2), U16.9 (VOUT2)
- new net: R55.1, U10.4 (EN)
- new net: D6.1 (K), R40.1
- new net: L6.1, U10.6 (LX)
- new net: D10.1 (K), R44.1
- new net +0.9V: C37.1, C47.1, L5.2, R37.1, U9.2 (OUT)
- new net +1.5V: C40.1, C48.1, L6.2, R35.1, U10.2 (OUT)
- new net +1V: C34.1, C46.1, L4.2, R32.1, U8.2 (OUT)
- new net +1V2: C44.1, U12.5 (VOUT)
- new net 0.9V_OK: R46.2, U9.3 (PG)
- new net 1.5V_OK: R36.2, U10.3 (PG)
- new net 1V_OK: R48.2, U8.3 (PG)
- new net 3.3V_OK: R45.2, U7.3 (PG)
- new net PO_1: R49.2, U13.3 (ON1)
- new net PO_2: R50.2, U13.5 (ON2)
- new net PO_3: R51.2, U14.3 (ON1)
- new net PO_4: R52.2, U14.5 (ON2)
- new net PO_5: U15.3 (ON1)
- new net PO_6: U15.5 (ON2)
- new net PO_7: U16.3 (ON1)
- new net PO_8: U16.5 (ON2)
- new net SY8843_3.3V_OUT: C29.1, C41.1, C42.1, C45.1, L3.2, R31.1, R36.1, R45.1, R46.1, R48.1, U11.1 (VIN), U12.1 (VIN), U13.1 (VIN1), U13.2 (VIN1), U13.4 (VBIAS), U7.2 (OUT)
Other:
- note added: "power good led"
