File: KiCad/Xeltri/Expansion_Port.kicad_sch (KiCad schematic)
At the start: 35 parts, among them J2 877159106, J3 HR911105A_C12074, U17 CH334P, U6 RTL8201F-VB-CG, Y1 25Mhz

Commit message: Rename the board to Xeltri and drop unused T113/old-selection files.
The KiCad project follows the rebrand; leftover T113 PDFs, the ESP32 stub, and unused HDMI/PMIC/inductor libraries are removed from the tree.

Co-authored-by: Cursor <cursoragent@cursor.com>
Parts:
- Y1: private KLC_S4.1 -> (none)
Changed lines of the file:
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@@
 		)
 		(instances
-			(project "TriCore-X"
+			(project "Xeltri"
 				(path "/b9ed8ff9-3a91-4311-b656-324fcf6f7e0c/0a747f2c-9f58-498b-af92-80cd731affd0"
 					(reference "C24")
@@
 		)
 		(instances
-			(project "TriCore-X"
+			(project "Xeltri"
 				(path "/b9ed8ff9-3a91-4311-b656-324fcf6f7e0c/0a747f2c-9f58-498b-af92-80cd731affd0"
 					(reference "#PWR07")
@@
 		)
 		(instances
-			(project "TriCore-X"
+			(project "Xeltri"
 				(path "/b9ed8ff9-3a91-4311-b656-324fcf6f7e0c/0a747f2c-9f58-498b-af92-80cd731affd0"
 					(reference "#PWR09")
@@
 		)
 		(instances
-			(project "TriCore-X"
+			(project "Xeltri"
 				(path "/b9ed8ff9-3a91-4311-b656-324fcf6f7e0c/0a747f2c-9f58-498b-af92-80cd731affd0"
 					(reference "R23")
@@
 		)
 		(instances
-			(project "TriCore-X"
+			(project "Xeltri"
 				(path "/b9ed8ff9-3a91-4311-b656-324fcf6f7e0c/0a747f2c-9f58-498b-af92-80cd731affd0"
 					(reference "D4")
@@
 		)
 		(instances
-			(project "TriCore-X"
+			(project "Xeltri"
 				(path "/b9ed8ff9-3a91-4311-b656-324fcf6f7e0c/0a747f2c-9f58-498b-af92-80cd731affd0"
 					(reference "R21")
@@
 		)
 		(instances
-			(project "TriCore-X"
+			(project "Xeltri"
 				(path "/b9ed8ff9-3a91-4311-b656-324fcf6f7e0c/0a747f2c-9f58-498b-af92-80cd731affd0"
 					(reference "R28")
@@
 		)
 		(instances
-			(project "TriCore-X"
+			(project "Xeltri"
 				(path "/b9ed8ff9-3a91-4311-b656-324fcf6f7e0c/0a747f2c-9f58-498b-af92-80cd731affd0"
 					(reference "C22")
@@
 		)
 		(instances
-			(project "TriCore-X"
+			(project "Xeltri"
 				(path "/b9ed8ff9-3a91-4311-b656-324fcf6f7e0c/0a747f2c-9f58-498b-af92-80cd731affd0"
 					(reference "#PWR036")
@@
 		)
 		(instances
-			(project "TriCore-X"
+			(project "Xeltri"
 				(path "/b9ed8ff9-3a91-4311-b656-324fcf6f7e0c/0a747f2c-9f58-498b-af92-80cd731affd0"
 					(reference "R25")
@@
 			)
 		)
-		(property private "KLC_S3.3" "The rectangle is not a symbol body but a graphical element"
-			(at 93.98 228.6 0)
-			(show_name yes)
-			(effects
-				(font
-					(size 1.27 1.27)
-				)
-				(hide yes)
-			)
-		)
-		(property private "KLC_S4.1" "Some pins are on 50mil grid to make the symbol small"
-			(at 93.98 231.14 0)
-			(show_name yes)
-			(effects
-				(font
-					(size 1.27 1.27)
-				)
-				(hide yes)
-			)
-		)
 		(pin "3"
 		)
@@
 		)
 		(instances
-			(project "TriCore-X"
+			(project "Xeltri"
 				(path "/b9ed8ff9-3a91-4311-b656-324fcf6f7e0c/0a747f2c-9f58-498b-af92-80cd731affd0"
 					(reference "R27")
@@
 		)
 		(instances
-			(project "TriCore-X"
+			(project "Xeltri"
 				(path "/b9ed8ff9-3a91-4311-b656-324fcf6f7e0c/0a747f2c-9f58-498b-af92-80cd731affd0"
 					(reference "R19")
@@
 		)
 		(instances
-			(project "TriCore-X"
+			(project "Xeltri"
 				(path "/b9ed8ff9-3a91-4311-b656-324fcf6f7e0c/0a747f2c-9f58-498b-af92-80cd731affd0"
 					(reference "C19")
@@
 		)
 		(instances
-			(project "TriCore-X"
+			(project "Xeltri"
 				(path "/b9ed8ff9-3a91-4311-b656-324fcf6f7e0c/0a747f2c-9f58-498b-af92-80cd731affd0"
 					(reference "R30")
@@
 		)
 		(instances
-			(project "TriCore-X"
+			(project "Xeltri"
 				(path "/b9ed8ff9-3a91-4311-b656-324fcf6f7e0c/0a747f2c-9f58-498b-af92-80cd731affd0"
 					(reference "#PWR03")
@@
 		)
 		(instances
-			(project "TriCore-X"
+			(project "Xeltri"
 				(path "/b9ed8ff9-3a91-4311-b656-324fcf6f7e0c/0a747f2c-9f58-498b-af92-80cd731affd0"
 					(reference "#PWR031")
@@
 		)
 		(instances
-			(project "TriCore-X"
+			(project "Xeltri"
 				(path "/b9ed8ff9-3a91-4311-b656-324fcf6f7e0c/0a747f2c-9f58-498b-af92-80cd731affd0"
 					(reference "#PWR042")
@@
 		)
 		(instances
-			(project "TriCore-X"
+			(project "Xeltri"
 				(path "/b9ed8ff9-3a91-4311-b656-324fcf6f7e0c/0a747f2c-9f58-498b-af92-80cd731affd0"
 					(reference "R18")
@@
 		)
 		(instances
-			(project "TriCore-X"
+			(project "Xeltri"
 				(path "/b9ed8ff9-3a91-4311-b656-324fcf6f7e0c/0a747f2c-9f58-498b-af92-80cd731affd0"
 					(reference "R22")
@@
 		)
 		(instances
-			(project "TriCore-X"
+			(project "Xeltri"
 				(path "/b9ed8ff9-3a91-4311-b656-324fcf6f7e0c/0a747f2c-9f58-498b-af92-80cd731affd0"
 					(reference "#PWR041")
@@
 		)
 		(instances
-			(project "TriCore-X"
+			(project "Xeltri"
 				(path "/b9ed8ff9-3a91-4311-b656-324fcf6f7e0c/0a747f2c-9f58-498b-af92-80cd731affd0"
 					(reference "R24")
@@
 		)
 		(instances
-			(project "TriCore-X"
+			(project "Xeltri"
 				(path "/b9ed8ff9-3a91-4311-b656-324fcf6f7e0c/0a747f2c-9f58-498b-af92-80cd731affd0"
 					(reference "C25")
@@
 		)
 		(instances
-			(project "TriCore-X"
+			(project "Xeltri"
 				(path "/b9ed8ff9-3a91-4311-b656-324fcf6f7e0c/0a747f2c-9f58-498b-af92-80cd731affd0"
 					(reference "R16")
@@
 		)
 		(instances
-			(project "TriCore-X"
+			(project "Xeltri"
 				(path "/b9ed8ff9-3a91-4311-b656-324fcf6f7e0c/0a747f2c-9f58-498b-af92-80cd731affd0"
 					(reference "C21")
@@
 		)
 		(instances
-			(project "TriCore-X"
+			(project "Xeltri"
 				(path "/b9ed8ff9-3a91-4311-b656-324fcf6f7e0c/0a747f2c-9f58-498b-af92-80cd731affd0"
 					(reference "#PWR04")
@@
 		)
 		(instances
-			(project "TriCore-X"
+			(project "Xeltri"
 				(path "/b9ed8ff9-3a91-4311-b656-324fcf6f7e0c/0a747f2c-9f58-498b-af92-80cd731affd0"
 					(reference "#PWR05")
@@
 		)
 		(instances
-			(project "TriCore-X"
+			(project "Xeltri"
 				(path "/b9ed8ff9-3a91-4311-b656-324fcf6f7e0c/0a747f2c-9f58-498b-af92-80cd731affd0"
 					(reference "C20")
@@
 		)
 		(instances
-			(project "TriCore-X"
+			(project "Xeltri"
 				(path "/b9ed8ff9-3a91-4311-b656-324fcf6f7e0c/0a747f2c-9f58-498b-af92-80cd731affd0"
 					(reference "#PWR040")
@@
 		)
 		(instances
-			(project "TriCore-X"
+			(project "Xeltri"
 				(path "/b9ed8ff9-3a91-4311-b656-324fcf6f7e0c/0a747f2c-9f58-498b-af92-80cd731affd0"
 					(reference "C23")
@@
 		)
 		(instances
-			(project "TriCore-X"
+			(project "Xeltri"
 				(path "/b9ed8ff9-3a91-4311-b656-324fcf6f7e0c/0a747f2c-9f58-498b-af92-80cd731affd0"
 					(reference "R17")
@@
 		)
 		(instances
-			(project "TriCore-X"
+			(project "Xeltri"
 				(path "/b9ed8ff9-3a91-4311-b656-324fcf6f7e0c/0a747f2c-9f58-498b-af92-80cd731affd0"
 					(reference "#PWR039")
@@
 		)
 		(instances
-			(project "TriCore-X"
+			(project "Xeltri"
 				(path "/b9ed8ff9-3a91-4311-b656-324fcf6f7e0c/0a747f2c-9f58-498b-af92-80cd731affd0"
 					(reference "R26")
@@
 		)
 		(instances
-			(project "TriCore-X"
+			(project "Xeltri"
 				(path "/b9ed8ff9-3a91-4311-b656-324fcf6f7e0c/0a747f2c-9f58-498b-af92-80cd731affd0"
 					(reference "R20")
@@
 		)
 		(instances
-			(project "TriCore-X"
+			(project "Xeltri"
 				(path "/b9ed8ff9-3a91-4311-b656-324fcf6f7e0c/0a747f2c-9f58-498b-af92-80cd731affd0"
 					(reference "C27")
@@
 		)
 		(instances
-			(project "TriCore-X"
+			(project "Xeltri"
 				(path "/b9ed8ff9-3a91-4311-b656-324fcf6f7e0c/0a747f2c-9f58-498b-af92-80cd731affd0"
 					(reference "R29")
@@
 		)
 		(instances
-			(project "TriCore-X"
+			(project "Xeltri"
 				(path "/b9ed8ff9-3a91-4311-b656-324fcf6f7e0c/0a747f2c-9f58-498b-af92-80cd731affd0"
 					(reference "C28")
@@
 		)
 		(instances
-			(project "TriCore-X"
+			(project "Xeltri"
 				(path "/b9ed8ff9-3a91-4311-b656-324fcf6f7e0c/0a747f2c-9f58-498b-af92-80cd731affd0"
 					(reference "C26")
@@
 		)
 		(instances
-			(project "TriCore-X"
+			(project "Xeltri"
 				(path "/b9ed8ff9-3a91-4311-b656-324fcf6f7e0c/0a747f2c-9f58-498b-af92-80cd731affd0"
 					(reference "#PWR038")
