File: KiCad/Xeltri/power.kicad_sch (KiCad schematic)
At the start: 110 parts, among them J1 PJ-035DH, Q1 AOD407, U10 SY8843QWC, U11 RT9013-18GB, U12 RT9013-12GB, U13 TPS22966DPUR, U14 TPS22966DPUR, U15 TPS22966DPUR, U16 TPS22966DPUR, U3 TPS56637RPAR, U4 TPS56637RPAR, U7 SY8843QWC, U8 SY8843QWC, U9 SY8843QWC

Commit message: Rename the board to Xeltri and drop unused T113/old-selection files.
The KiCad project follows the rebrand; leftover T113 PDFs, the ESP32 stub, and unused HDMI/PMIC/inductor libraries are removed from the tree.

Co-authored-by: Cursor <cursoragent@cursor.com>
Parts:
- added R59, R60: 0R, Resistor_SMD:R_0402_1005Metric, symbol Device:R
- C1, C11, C12, C2: footprint Capacitor_SMD:C_0402_1005Metric -> Capacitor_SMD:C_1210_3225Metric
- C13, C3: value 0.1uF -> 100nF; footprint Capacitor_SMD:C_0402_1005Metric -> Capacitor_SMD:C_0805_2012Metric
Connections:
- net at L2.1, U4.6 (SW): now also R60.2; no longer C14.1
- net at U4.7 (BOOT): now also C14.1; no longer C14.2
- net at L1.1, U3.6 (SW): now also R59.2; no longer C4.1
- net at U3.7 (BOOT): now also C4.1; no longer C4.2
- new net: C4.2, R59.1
- new net: C14.2, R60.1
Other:
- moved on the sheet: C14, C4
